File: Badge.brd (EAGLE design)
At the start: 160 x 100 mm, 71 parts, among them IC1 ATMEGA328P-AU, IC2 ATSAMD11C14A-SSNT, IC3 BME280, IC4 BNO055, IC5 MCP79400-I_SN, J1 54819-0572, J2 FTS-105-01-L-DV-P-TR, J3 3002, SW1 B3FS-1000P, SW2 B3FS-1000P, SW3 B3FS-1000P, SW4 B3FS-1000P, SW5 B3FS-1000P, Y1 ABM3-16.000MHZ-B2-T, Y2 MC-306_32.7680K-E3_ROHS, Y3 MC-306_32.7680K-E3_ROHS

Commit message: Added Power and LEDs
Also added a new library.
Parts:
- added C25, C26, C28: 0.1 uF, rcl:C0603K
- added C27, C29: 22uF 16V 4.3mm, Badge_v202004081200_Eagle_Library_regex:CAPAE430X550L180X65N
- added C30: 10u, rcl:C0805K
- added C31, C32, C33, C34: 0.1u, rcl:C0603K
- added C35: EEE1VA2R2NR, SamacSys_Parts:CAPAE430X550N
- added D2, D3, D4, D5: WS2812B, Badge_v202004081200_Eagle_Library_regex:WS2812B
- added IC6: MIC5219-5.0YM5-TR, Badge_v202004081200_Eagle_Library_regex:SOT23-5P95_280X145L45X37N
- added IC7: MIC5219-3.3YM5-TR, Badge_v202004081200_Eagle_Library_regex:SOT23-5P95_280X145L45X37N
- added J4: DNP, Badge_v202004081200_Eagle_Library_regex:BATIN
- added LED1: APA3010CGCK-GX, SamacSys_Parts:APA3010ZGCGX
- added LS1: AST-03008MR-R, Badge_v202004081200_Eagle_Library_regex:PUIAUDIO_AST-03008MR-R
- added Q1: BSS138LT7G, SamacSys_Parts:SOT96P237X111-3N
- added R21, R22: 100k, rcl:R0603
- added R23: 0, rcl:R0603
- added R24, R25: 22, Badge:R0603
- added SW6: JS202011SCQN, Badge_v202004081200_Eagle_Library_regex:JS202011SCQN
- added TP11, TP12, TP13, TP14: PTR1PAD1-20, testpad:P1-20
- Y2, Y3: value MC-306_32.7680K-E3_ROHS -> 32.768 kHz; device SamacSys_Parts:MC306327680KE3ROHS -> Badge_v202004081200_Eagle_Library_regex:XTAL960X406X315
- moved Y2 290.3 mm to (-138.4, -494.0)
- moved Y3 181.3 mm to (-138.4, -488.9)
Connections:
- new net +5V: C27.1, C30.1, C31.1, C32.1, C33.1, C34.1, D2.1, D3.1, D4.1, D5.1, IC6.5, IC7.1, IC7.3, R23.1, TP11.TP
- new net +5V1: C29.1, IC7.5, TP13.TP
- new net N$18: J4.1, SW6.2, SW6.5
- new net N$25: D3.2, D4.4
- new net N$26: D4.2, D5.4
- new net N$27: C25.1, IC6.1, R21.2, SW6.3, SW6.6
- new net N$28: IC6.3, Q1.3, R21.1, TP12.TP
- new net N$29: D2.4, R24.2
- new net VCC: Q1.1, R22.2, R23.2
- net ADDR_LED: now also R24.1, TP14.TP
- net BUZZER: now also C35.1
- net GND: now also C25.2, C26.2, C27.2, C28.2, C29.2, C30.2, C31.2, C32.2, C33.2, C34.2, D3.3, D4.3, D5.3, IC6.2, IC7.2, J2.3, J2.5, J4.2, LS1.2, Q1.2, R22.1, R25.1; no longer Y2.2, Y2.3, Y3.2, Y3.3
- net LED_INDICATOR: now also LED1.2
- net N$10: now also C35.2, LS1.1; no longer R5.1, R6.2
- net N$11: now also C28.1, IC7.4; no longer J2.3, J2.5
- net N$12: now also LED1.1, R25.2; no longer R7.1, R8.2
- net N$14: now also R10.2, R9.1
- net N$15: now also D2.2, D3.4; no longer R10.2, R9.1
- net N$16: now also Y2.1; no longer Y2.4
- net N$17: now also Y2.2; no longer Y2.1
- net N$23: now also Y3.2; no longer Y3.4
- net N$5: now also C26.1, IC6.4; no longer R3.1, R4.2
- net N$6: now also R5.1, R6.2
- net N$7: now also R7.1, R8.2
- net N$8: now also R3.1, R4.2
