File: Badge.sch (EAGLE design)
At the start: 71 parts, among them IC1 ATMEGA328P-AU, IC2 ATSAMD11C14A-SSNT, IC3 BME280, IC4 BNO055, IC5 MCP79400-I_SN, J1 54819-0572, J2 FTS-105-01-L-DV-P-TR, J3 3002, SW1 B3FS-1000P, SW2 B3FS-1000P, SW3 B3FS-1000P, SW4 B3FS-1000P, SW5 B3FS-1000P, Y1 ABM3-16.000MHZ-B2-T, Y2 MC-306_32.7680K-E3_ROHS, Y3 MC-306_32.7680K-E3_ROHS

Commit message: Added Power and LEDs
Also added a new library.
Parts:
- added C25, C26, C28: 0.1 uF, rcl:C-USC0603K
- added C27, C29: 22uF 16V 4.3mm, Badge_v202004081200_Eagle_Library_regex:22_UF_16V_4.3MM
- added C30: 10u, rcl:C-USC0805K
- added C31, C32, C33, C34: 0.1u, rcl:C-USC0603K
- added C35: EEE1VA2R2NR, SamacSys_Parts:EEE1VA2R2NR
- added D2, D3, D4, D5: WS2812B, Badge_v202004081200_Eagle_Library_regex:WS2812B
- added IC6: MIC5219-5.0YM5-TR, Badge_v202004081200_Eagle_Library_regex:MIC5219-5.0YM5-TR
- added IC7: MIC5219-3.3YM5-TR, Badge_v202004081200_Eagle_Library_regex:MIC5219-3.3YM5-TR
- added J4: DNP, Badge_v202004081200_Eagle_Library_regex:BAT_CONNECTOR
- added LED1: APA3010CGCK-GX, SamacSys_Parts:APA3010CGCK-GX
- added LS1: AST-03008MR-R, Badge_v202004081200_Eagle_Library_regex:AST-03008MR-R
- added Q1: BSS138LT7G, SamacSys_Parts:BSS138LT7G
- added R21, R22: 100k, rcl:R-US_R0603
- added R23: 0, rcl:R-US_R0603
- added R24, R25: 22, Badge:R-US_R0603
- added SW6: JS202011SCQN, Badge_v202004081200_Eagle_Library_regex:JS202011SCQN
- added TP11, TP12, TP13, TP14: PTR1PAD1-20, testpad:PTR1PAD1-20
- Y2, Y3: value MC-306_32.7680K-E3_ROHS -> 32.768 kHz; device SamacSys_Parts:MC-306_32.7680K-E3_ROHS -> Badge_v202004081200_Eagle_Library_regex:MC-405
Connections:
- new net +5V: C27.PLUS, C30.1, C31.1, C32.1, C33.1, C34.1, D2.1, D3.1, D4.1, D5.1, IC6.OUT, IC7.EN, IC7.IN, R23.1, TP11.TP
- new net +5V1: C29.PLUS, IC7.OUT, TP13.TP
- new net N$18: J4.1, SW6.2, SW6.5
- new net N$25: D3.2, D4.4
- new net N$26: D4.2, D5.4
- new net N$27: C25.1, IC6.IN, R21.2, SW6.3, SW6.6
- new net N$28: IC6.EN, Q1.D, R21.1, TP12.TP
- new net N$29: D2.4, R24.2
- new net VCC: Q1.G, R22.2, R23.2
- net ADDR_LED: now also R24.1, TP14.TP
- net BUZZER: now also C35.+
- net GND: now also C25.2, C26.2, C27.MINUS, C28.2, C29.MINUS, C30.2, C31.2, C32.2, C33.2, C34.2, D3.3, D4.3, D5.3, IC6.GND, IC7.GND, J2.3, J2.5, J4.2, LS1.2, Q1.S, R22.1, R25.1; no longer Y2.GND_1, Y2.GND_2, Y3.GND_1, Y3.GND_2
- net LED_INDICATOR: now also LED1.A
- net N$10: now also C35.-, LS1.1; no longer R5.1, R6.2
- net N$11: now also C28.1, IC7.BYP; no longer J2.3, J2.5
- net N$12: now also LED1.K, R25.2; no longer R7.1, R8.2
- net N$14: now also R10.2, R9.1
- net N$15: now also D2.2, D3.4; no longer R10.2, R9.1
- net N$16: now also Y2.1; no longer Y2.CRYSTAL_2
- net N$17: now also Y2.2; no longer Y2.CRYSTAL_1
- net N$23: now also Y3.2; no longer Y3.CRYSTAL_2
- net N$24: now also Y3.1; no longer Y3.CRYSTAL_1
- net N$5: now also C26.1, IC6.BYP; no longer R3.1, R4.2
- net N$6: now also R5.1, R6.2
- net N$7: now also R7.1, R8.2
- net N$8: now also R3.1, R4.2
Other:
- note added: "LED/BUZZER"
- note added: "Power"
- note added: "RTC"
